File: hardware/address_bus.kicad_sch (KiCad schematic)
At the start: 17 parts, among them Q7 BC557, Q8 BC557, U2 74LS06N, U5 74HC595, U6 74HC595, U7 74HC595

Commit message: Rev.F. Update project
Other:
- note added: "1W"
Changed lines of the file:
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@@
   (title_block
     (title "USB Flash/EPROM Programmer")
-    (date "2022-06-01")
+    (date "2022-07-06")
     (rev "v0.1.0 rev.F")
     (company "Robson Martins")
@@
   (wire (pts (xy 124.46 114.3) (xy 93.98 114.3))
     (stroke (width 0) (type default) (color 0 0 0 0))
+  )
+  (text "1W" (at 184.8438 93.0288 0)
+    (effects (font (size 1.27 1.27)) (justify left bottom))
+  )
+  (text "1W" (at 184.8438 138.7215 0)
+    (effects (font (size 1.27 1.27)) (justify left bottom))
   )
   (label "A18INT" (at 130.81 129.54 0)
@@
       (effects (font (size 1.27 1.27)) hide)
     )
+    (pin "1")
+    (pin "2")
+    (pin "3")
+    (pin "4")
+    (pin "5")
+    (pin "6")
     (pin "8")
     (pin "9")
+    (pin "10")
+    (pin "11")
+    (pin "12")
+    (pin "13")
+    (pin "14")
+    (pin "7")
   )
   (symbol (lib_id "74xx:74LS06N") (at 157.48 121.92 0) (unit 5)
@@
       (effects (font (size 1.27 1.27)) hide)
     )
+    (pin "1")
+    (pin "2")
+    (pin "3")
+    (pin "4")
+    (pin "5")
+    (pin "6")
+    (pin "8")
+    (pin "9")
     (pin "10")
     (pin "11")
+    (pin "12")
+    (pin "13")
+    (pin "14")
+    (pin "7")
   )
   (symbol (lib_id "Device:R") (at 170.18 76.2 90) (unit 1)
