File: hardware/address_bus.kicad_sch (KiCad schematic)
At the start: 17 parts, among them Q7 BC557, Q8 BC557, U2 74LS06N, U5 74HC595, U6 74HC595, U7 74HC595

Commit message: 0.3.rev.A. Created new main pcb
Parts:
- C11, C12, C13: footprint Capacitor_THT:C_Disc_D6.0mm_W2.5mm_P5.00mm -> Capacitor_THT:C_Disc_D5.0mm_W2.5mm_P5.00mm
- D12, D13: footprint Diode_THT:D_DO-35_SOD27_P7.62mm_Horizontal -> Diode_THT:D_DO-34_SOD68_P7.62mm_Horizontal
- R23, R24, R25, R26, R27, R28: footprint Resistor_THT:R_Axial_DIN0207_L6.3mm_D2.5mm_P10.16mm_Horizontal -> Resistor_THT:R_Axial_DIN0204_L3.6mm_D1.6mm_P7.62mm_Horizontal
