File: hardware/control_signals.kicad_sch (KiCad schematic)
At the start: 25 parts, among them Q10 BC557, Q11 BC557, Q12 BC547, Q9 BC557, U8 74LS06N

Commit message: Rev.F. Update project
Connections:
- net ~{CE}: now also R40.1; no longer R40.2
- net at Q11.1 (C): now also R40.2; no longer R40.1
Other:
- note added: "1W"
- moved on the sheet: R40
Changed lines of the file:
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@@
   (title_block
     (title "USB Flash/EPROM Programmer")
-    (date "2022-06-01")
+    (date "2022-07-06")
     (rev "v0.1.0 rev.F")
     (company "Robson Martins")
@@
   (junction (at 147.32 90.17) (diameter 0) (color 0 0 0 0)
   )
-  (junction (at 232.41 90.17) (diameter 0) (color 0 0 0 0)
-  )
   (junction (at 68.58 118.11) (diameter 0) (color 0 0 0 0)
   )
@@
   (junction (at 139.7 48.26) (diameter 0) (color 0 0 0 0)
   )
+  (junction (at 222.25 92.71) (diameter 0) (color 0 0 0 0)
+  )
   (junction (at 139.7 102.87) (diameter 0) (color 0 0 0 0)
   )
@@
     (stroke (width 0) (type default) (color 0 0 0 0))
   )
-  (wire (pts (xy 222.25 90.17) (xy 223.52 90.17))
-    (stroke (width 0) (type default) (color 0 0 0 0))
-  )
-  (wire (pts (xy 222.25 82.55) (xy 222.25 90.17))
-    (stroke (width 0) (type default) (color 0 0 0 0))
-  )
   (wire (pts (xy 68.58 107.95) (xy 86.36 107.95))
     (stroke (width 0) (type default) (color 0 0 0 0))
@@
     (stroke (width 0) (type default) (color 0 0 0 0))
   )
-  (wire (pts (xy 232.41 92.71) (xy 232.41 90.17))
-    (stroke (width 0) (type default) (color 0 0 0 0))
-  )
   (wire (pts (xy 58.42 55.88) (xy 68.58 55.88))
     (stroke (width 0) (type default) (color 0 0 0 0))
@@
     (stroke (width 0) (type default) (color 0 0 0 0))
   )
-  (wire (pts (xy 231.14 90.17) (xy 232.41 90.17))
-    (stroke (width 0) (type default) (color 0 0 0 0))
-  )
   (wire (pts (xy 68.58 109.22) (xy 68.58 107.95))
     (stroke (width 0) (type default) (color 0 0 0 0))
@@
     (stroke (width 0) (type default) (color 0 0 0 0))
   )
+  (wire (pts (xy 222.25 90.17) (xy 222.25 92.71))
+    (stroke (width 0) (type default) (color 0 0 0 0))
+  )
   (wire (pts (xy 58.42 118.11) (xy 68.58 118.11))
     (stroke (width 0) (type default) (color 0 0 0 0))
@@
     (stroke (width 0) (type default) (color 0 0 0 0))
   )
-  (wire (pts (xy 232.41 90.17) (xy 232.41 88.9))
+  (wire (pts (xy 232.41 88.9) (xy 232.41 92.71))
     (stroke (width 0) (type default) (color 0 0 0 0))
   )
@@
   (wire (pts (xy 138.43 102.87) (xy 139.7 102.87))
     (stroke (width 0) (type default) (color 0 0 0 0))
+  )
+  (text "1W" (at 234.4573 102.2384 0)
+    (effects (font (size 1.27 1.27)) (justify left bottom))
+  )
+  (text "1W" (at 149.2446 127.2591 0)
+    (effects (font (size 1.27 1.27)) (justify left bottom))
+  )
+  (text "1W" (at 149.4538 65.3726 0)
+    (effects (font (size 1.27 1.27)) (justify left bottom))
   )
   (global_label "VPP_RAW" (shape passive) (at 234.95 64.77 0) (fields_autoplaced)
@@
     (pin "1")
     (pin "2")
+    (pin "3")
+    (pin "4")
+    (pin "5")
+    (pin "6")
+    (pin "8")
+    (pin "9")
+    (pin "10")
+    (pin "11")
+    (pin "12")
+    (pin "13")
+    (pin "14")
+    (pin "7")
   )
   (symbol (lib_id "Device:R") (at 134.62 48.26 90) (unit 1)
@@
       (effects (font (size 1.27 1.27)) hide)
     )
+    (pin "1")
+    (pin "2")
     (pin "3")
     (pin "4")
+    (pin "5")
+    (pin "6")
+    (pin "8")
+    (pin "9")
+    (pin "10")
+    (pin "11")
+    (pin "12")
+    (pin "13")
+    (pin "14")
+    (pin "7")
   )
   (symbol (lib_id "74xx:74LS06N") (at 121.92 102.87 0) (unit 3)
@@
       (effects (font (size 1.27 1.27)) hide)
     )
+    (pin "1")
+    (pin "2")
+    (pin "3")
+    (pin "4")
     (pin "5")
     (pin "6")
+    (pin "8")
+    (pin "9")
+    (pin "10")
+    (pin "11")
+    (pin "12")
+    (pin "13")
+    (pin "14")
+    (pin "7")
   )
   (symbol (lib_id "Device:R") (at 134.62 102.87 90) (unit 1)
@@
       (effects (font (size 1.27 1.27)) hide)
     )
+    (pin "1")
+    (pin "2")
+    (pin "3")
+    (pin "4")
+    (pin "5")
+    (pin "6")
     (pin "8")
     (pin "9")
+    (pin "10")
+    (pin "11")
+    (pin "12")
+    (pin "13")
+    (pin "14")
+    (pin "7")
   )
   (symbol (lib_id "Diode:1N4148") (at 152.4 113.03 180) (unit 1)
@@
       (effects (font (size 1.27 1.27)) hide)
     )
+    (pin "1")
+    (pin "2")
+    (pin "3")
+    (pin "4")
+    (pin "5")
+    (pin "6")
+    (pin "8")
+    (pin "9")
     (pin "10")
     (pin "11")
+    (pin "12")
+    (pin "13")
+    (pin "14")
+    (pin "7")
   )
   (symbol (lib_id "Device:R") (at 209.55 77.47 90) (unit 1)
@@
     (pin "2")
   )
-  (symbol (lib_id "Device:R") (at 227.33 90.17 90) (unit 1)
-    (in_bom yes) (on_board yes)
-    (property "Reference" "R40" (id 0) (at 227.33 84.9122 90))
-    (property "Value" "100R" (id 1) (at 227.33 87.2236 90))
-    (property "Footprint" "Resistor_THT:R_Axial_DIN0207_L6.3mm_D2.5mm_P10.16mm_Horizontal" (id 2) (at 227.33 91.948 90)
-      (effects (font (size 1.27 1.27)) hide)
-    )
-    (property "Datasheet" "~" (id 3) (at 227.33 90.17 0)
+  (symbol (lib_id "Device:R") (at 222.25 86.36 180) (unit 1)
+    (in_bom yes) (on_board yes)
+    (property "Reference" "R40" (id 0) (at 217.845 85.1036 0))
+    (property "Value" "100R" (id 1) (at 217.4564 87.1117 0))
+    (property "Footprint" "Resistor_THT:R_Axial_DIN0207_L6.3mm_D2.5mm_P10.16mm_Horizontal" (id 2) (at 224.028 86.36 90)
+      (effects (font (size 1.27 1.27)) hide)
+    )
+    (property "Datasheet" "~" (id 3) (at 222.25 86.36 0)
       (effects (font (size 1.27 1.27)) hide)
     )
@@
       (effects (font (size 1.27 1.27)) hide)
     )
+    (pin "1")
+    (pin "2")
+    (pin "3")
+    (pin "4")
+    (pin "5")
+    (pin "6")
+    (pin "8")
+    (pin "9")
+    (pin "10")
+    (pin "11")
+    (pin "12")
+    (pin "13")
     (pin "14")
     (pin "7")
