File: hardware/control_signals.kicad_sch (KiCad schematic)
At the start: 25 parts, among them Q10 BC557, Q11 BC557, Q12 BC547, Q9 BC557, U8 74LS06N

Commit message: 0.3.rev.A. Created new main pcb
Parts:
- C14: footprint Capacitor_THT:C_Disc_D6.0mm_W2.5mm_P5.00mm -> Capacitor_THT:C_Disc_D5.0mm_W2.5mm_P5.00mm
- D14, D15, D16, D17, D18: footprint Diode_THT:D_DO-35_SOD27_P7.62mm_Horizontal -> Diode_THT:D_DO-34_SOD68_P7.62mm_Horizontal
- R29, R30, R31, R32, R33, R34, R35, R36, R37, R38, R39, R40, R41, R42: footprint Resistor_THT:R_Axial_DIN0207_L6.3mm_D2.5mm_P10.16mm_Horizontal -> Resistor_THT:R_Axial_DIN0204_L3.6mm_D1.6mm_P7.62mm_Horizontal
