File: hardware/cpu.kicad_sch (KiCad schematic)
At the start: 4 parts, among them U3 Pico, U4 74HC595

Commit message: 0.3.rev.A. Created new main pcb
Parts:
- C10: footprint Capacitor_THT:C_Disc_D6.0mm_W2.5mm_P5.00mm -> Capacitor_THT:C_Disc_D5.0mm_W2.5mm_P5.00mm
- R22: footprint Resistor_THT:R_Axial_DIN0207_L6.3mm_D2.5mm_P10.16mm_Horizontal -> Resistor_THT:R_Axial_DIN0204_L3.6mm_D1.6mm_P7.62mm_Horizontal
