File: hardware/data_bus.kicad_sch (KiCad schematic)
At the start: 11 parts, among them Q13 BC547, U10 74HC595, U11 74HC165, U12 74HC165, U9 74HC595

Commit message: 0.3.rev.A. Created new main pcb
Parts:
- C15, C16, C17, C18: footprint Capacitor_THT:C_Disc_D6.0mm_W2.5mm_P5.00mm -> Capacitor_THT:C_Disc_D5.0mm_W2.5mm_P5.00mm
- R43, R44: footprint Resistor_THT:R_Axial_DIN0207_L6.3mm_D2.5mm_P10.16mm_Horizontal -> Resistor_THT:R_Axial_DIN0204_L3.6mm_D1.6mm_P7.62mm_Horizontal
