File: hardware/serial_bus.kicad_sch (KiCad schematic)
At the start: 15 parts, among them Q14 BC547, Q15 BC547, Q16 BC547, U2 74LS06N, U8 74LS06N

Commit message: 0.3.rev.A. Created new main pcb
Parts:
- D19, D20: footprint Diode_THT:D_DO-41_SOD81_P10.16mm_Horizontal -> Diode_THT:D_DO-35_SOD27_P7.62mm_Horizontal
- R45, R46, R47, R48, R49, R50, R51: footprint Resistor_THT:R_Axial_DIN0207_L6.3mm_D2.5mm_P10.16mm_Horizontal -> Resistor_THT:R_Axial_DIN0204_L3.6mm_D1.6mm_P7.62mm_Horizontal
- R52: footprint Resistor_THT:R_Axial_DIN0309_L9.0mm_D3.2mm_P15.24mm_Horizontal -> Resistor_THT:R_Axial_DIN0207_L6.3mm_D2.5mm_P10.16mm_Horizontal
