File: hardware/usbflashprog.kicad_sch (KiCad schematic)
At the start: 8 parts, among them J2 Parallel Adapter, J3 Serial Adapter, U1 MT3608 Module

Commit message: 0.3.rev.A. Created new main pcb
Parts:
- C3: footprint Capacitor_THT:C_Disc_D6.0mm_W2.5mm_P5.00mm -> Capacitor_THT:C_Disc_D5.0mm_W2.5mm_P5.00mm
- R1: footprint Resistor_THT:R_Axial_DIN0207_L6.3mm_D2.5mm_P10.16mm_Horizontal -> Resistor_THT:R_Axial_DIN0204_L3.6mm_D1.6mm_P7.62mm_Horizontal
