File: hardware/vpp_generator.kicad_sch (KiCad schematic)
At the start: 17 parts, among them Q5 TIP120, Q6 BC327, U2 74LS06N

Commit message: 0.3.rev.A. Created new main pcb
Parts:
- C7, C9: footprint Capacitor_THT:C_Disc_D6.0mm_W2.5mm_P5.00mm -> Capacitor_THT:C_Disc_D5.0mm_W2.5mm_P5.00mm
- D11: footprint Diode_THT:D_DO-35_SOD27_P7.62mm_Horizontal -> Diode_THT:D_DO-34_SOD68_P7.62mm_Horizontal
- R15, R16, R17, R18, R19, R20, R21: footprint Resistor_THT:R_Axial_DIN0207_L6.3mm_D2.5mm_P10.16mm_Horizontal -> Resistor_THT:R_Axial_DIN0204_L3.6mm_D1.6mm_P7.62mm_Horizontal
